Commit message: elektron_control configuration, add elektron_world, elektron_navigation first commit

File: elektron_description/robots/elektron_laser_NoTower.urdf.xacro (robot description, xacro)
@@ -191,16 +191,13 @@
 	</gazebo>
   <gazebo>
-    <controller:gazebo_ros_controller_manager name="gazebo_ros_controller_manager" plugin="libgazebo_ros_controller_manager.so">
+  <plugin name="gazebo_ros_control" filename="libgazebo_ros_control.so">
+    <robotNamespace>/elektron</robotNamespace>
+<!--<robotSimType>gazebo_ros_control/DefaultRobotHWSim</robotSimType> -->
+  </plugin>
+   <!-- <controller:gazebo_ros_controller_manager name="gazebo_ros_controller_manager" plugin="libgazebo_ros_controller_manager.so">
       <alwaysOn>true</alwaysOn>
       <updateRate>1000.0</updateRate>
       <interface:audio name="gazebo_ros_controller_manager_dummy_iface" />
     </controller:gazebo_ros_controller_manager>
-  </gazebo>
-<gazebo>
-  <plugin name="gazebo_ros_control" filename="libgazebo_ros_control.so">
-    <robotNamespace>/elektron</robotNamespace>
-<robotSimType>gazebo_ros_control/DefaultRobotHWSim</robotSimType>
-  </plugin>
-<!--
  <transmission name="tran_state_right_wheel_joint">
     <type>joint_state_controller/JointStateController</type>
@@ -223,4 +220,6 @@
     </actuator>
   </transmission>
+-->
+</gazebo>
   <transmission name="tran_effort_left_wheel_joint">
     <type>effort_controllers/JointPositionController</type>
@@ -228,5 +227,5 @@
       <hardwareInterface>EffortJointInterface</hardwareInterface>
     </joint>
-    <actuator name="motorbase_link_left_wheel_joint">
+    <actuator name="motor_base_link_left_wheel_joint">
       <hardwareInterface>EffortJointInterface</hardwareInterface>
       <mechanicalReduction>1</mechanicalReduction>
@@ -238,11 +237,27 @@
       <hardwareInterface>EffortJointInterface</hardwareInterface>
     </joint>
-    <actuator name="motorbase_link_right_wheel_joint">
+    <actuator name="motor_base_link_right_wheel_joint">
       <hardwareInterface>EffortJointInterface</hardwareInterface>
       <mechanicalReduction>1</mechanicalReduction>
     </actuator>
   </transmission>
--->
-</gazebo>
+  <transmission name="tran_vel_left_wheel_joint">
+    <type>effort_controllers/JointVelocityController</type>
+    <joint name="base_link_left_wheel_joint">
+      <hardwareInterface>VelocityJointInterface</hardwareInterface>
+    </joint>
+    <actuator name="motor_base_link_left_wheel_joint">
+      <hardwareInterface>VelocityJointInterface</hardwareInterface>
+    </actuator>
+  </transmission>
+  <transmission name="tran_vel_right_wheel_joint">
+    <type>effort_controllers/JointVelocityController</type>
+    <joint name="base_link_right_wheel_joint">
+      <hardwareInterface>VelocityJointInterface</hardwareInterface>
+    </joint>
+    <actuator name="motor_base_link_right_wheel_joint">
+      <hardwareInterface>VelocityJointInterface</hardwareInterface>
+    </actuator>
+  </transmission>
 	<gazebo>
 		<controller:gazebo_ros_p3d name="p3d_base_controller" plugin="libgazebo_ros_p3d.so">
@@ -257,5 +272,4 @@
 			<interface:position name="p3d_base_position"/>
 		</controller:gazebo_ros_p3d>
-		<!--
 		<controller:differential_position2d name="controller1">
 			<update>100</update>
@@ -278,5 +292,4 @@
 			<interface:position name="p3d_base_position"/>
 		</controller:gazebo_ros_p3d>
-		-->
 		<controller:gazebo_ros_imu name="imu_controller" plugin="libgazebo_ros_imu.so">
 			<alwaysOn>true</alwaysOn>
@@ -285,5 +298,5 @@
 			<topicName>body_pose_ground_truth</topicName>
 			<xyzOffsets>25.7 25.7 0</xyzOffsets>
-			<!-- option to initialize odometry for fake localization-->
+			 option to initialize odometry for fake localization
 			<rpyOffsets>0 0 0</rpyOffsets>
 			<gaussianNoise>0.5</gaussianNoise>
