Commit message: fix head_rgb, set head_rgb as default, add top_kinect to tower

File: elektron_description/robots/elektron_Laser_Tower-rgb.urdf.xacro (robot description, xacro)
@@ -5,5 +5,5 @@
 	xmlns:interface="http://playerstage.sourceforge.net/gazebo/xmlschema/#interface">
 	<property name="M_PI" value="3.14159"/>
-	<property name="elektron_control_input" value="pid" /> <!-- diff_drive_controller | pid -->
+	<property name="elektron_control_input" value="1" /> <!-- 0 = diff_drive_controller | 1 = pid -->
 	<property name="base_size_x" value="0.38" />
 	<property name="base_size_y" value="0.28" />
@@ -47,6 +47,6 @@
 		</collision>
 	</link>
-	<!-- WHEELS MACRO -->
-	<xacro:macro name="erratic_wheel" params="suffix parent reflect offset m mimic">
+<!-- WHEELS MACRO -->
+	<xacro:macro name="erratic_wheel" params="suffix parent reflect offset m mimic mimic_wheel">
 			<joint name="${parent}_${suffix}_wheel_joint" type="continuous">
 				<origin xyz="${offset} ${reflect*caster_wheel_offset_y} ${wheel_radius}" rpy="0	0 0"/>
@@ -58,9 +58,6 @@
 				<child link="${parent}_${suffix}_wheel_link" />
 	 			<dynamics damping="0.0" friction="0.0"/>
-	 			<xacro:if value="${mimic == 'left'}">
-		 			<mimic joint="${parent}_${mimic}_wheel_joint"/>
-				</xacro:if>
-	 			<xacro:if value="${mimic == 'right'}">
-		 			<mimic joint="${parent}_${mimic}_wheel_joint"/>
+	 			<xacro:if value="${mimic}">
+		 			<mimic joint="${parent}_${mimic_wheel}_wheel_joint"/>
 				</xacro:if>
 			</joint>
@@ -96,11 +93,11 @@
 	</xacro:macro>
 	<!-- WHEELS DEFINITION -->
-	<xacro:erratic_wheel suffix="left" parent="base_link" reflect="1" offset="0" m="0.900" mimic="none"/>
-	<xacro:erratic_wheel suffix="left_front" parent="base_link" reflect="1" offset="0.15" m="0" mimic="left"/>
-	<xacro:erratic_wheel suffix="left_rear" parent="base_link" reflect="1" offset="-0.15" m="0" mimic="left"/>
-	<xacro:erratic_wheel suffix="right" parent="base_link" reflect="-1" offset="0" m="0.900" mimic="none"/>
+	<xacro:erratic_wheel suffix="left" parent="base_link" reflect="1" offset="0" m="0.900" mimic="0" mimic_wheel="left"/>
+	<xacro:erratic_wheel suffix="left_front" parent="base_link" reflect="1" offset="0.15" m="0" mimic="1" mimic_wheel="left"/>
+	<xacro:erratic_wheel suffix="left_rear" parent="base_link" reflect="1" offset="-0.15" m="0" mimic="1" mimic_wheel="left"/>
+	<xacro:erratic_wheel suffix="right" parent="base_link" reflect="-1" offset="0" m="0.900" mimic="0" mimic_wheel="left"/>
 	<xacro:erratic_wheel suffix="right_front" parent="base_link" reflect="-1" offset="0.15"
-		m="0" mimic="right"/>
-	<xacro:erratic_wheel suffix="right_rear" parent="base_link" reflect="-1" offset="-0.15"	m="0" mimic="right"/>
+		m="0" mimic="1" mimic_wheel="right" />
+	<xacro:erratic_wheel suffix="right_rear" parent="base_link" reflect="-1" offset="-0.15"	m="0" mimic="1" mimic_wheel="right"/>
 <!-- ADD KINECT -->
     <joint name="bottom_kinect_joint" type="fixed">
@@ -112,11 +109,11 @@
 	<sensor_kinect parent="bottom_kinect_link" id="bottom"/>
 	<!-- ADD TOWER -->
-	<elektron_tower parent="base_link" camera_type="rgb_camera" id="1"/> <!-- camera_type avaliable: kinect | rgb_camera -->
+	<elektron_tower parent="base_link" camera_type="1" id="1"/> <!-- camera_type avaliable: 1 = kinect | 0 = rgb_camera -->
 	<tower_PID_control_gazebo/>
 	<!-- SET gazebo-ROS CONTROL -->
-	<xacro:if value="${elektron_control_input == 'pid'}">
+	<xacro:if value="${elektron_control_input}">
 		<elektron_PID_control_gazebo/>
 	</xacro:if>
-	<xacro:if value="${elektron_control_input == 'diff_drive_controller'}">
+	<xacro:unless value="${elektron_control_input}">
 		<gazebo>
 		<plugin name="differential_drive_controller" filename="libgazebo_ros_diff_drive.so">
@@ -134,4 +131,4 @@
 		</plugin>
 	</gazebo>
-	</xacro:if>
+	</xacro:unless>
 </robot>

File: elektron_description/urdf/elektron_properties.urdf.xacro (robot description, xacro)
@@ -25,9 +25,15 @@
 	<property name="kinect_op" value="0" />
 	<property name="kinect_oy" value="0" />
-  <property name="head_base_px" value="0.1" />
-  <property name="head_base_py" value="0.0" />
-  <property name="head_base_pz" value="0.75"/>
-  <property name="head_base_or" value="0" />
-  <property name="head_base_op" value="0" />
-  <property name="head_base_oy" value="0" />
+	<property name="head_base_px" value="0.1" />
+	<property name="head_base_py" value="0.0" />
+	<property name="head_base_pz" value="0.75"/>
+	<property name="head_base_or" value="0" />
+	<property name="head_base_op" value="0" />
+	<property name="head_base_oy" value="0" />
+	<property name="high_kinect_base_px" value="0" />
+	<property name="high_kinect_base_py" value="0" />
+	<property name="high_kinect_base_pz" value="1.2" />
+	<property name="high_kinect_base_or" value="0" />
+	<property name="high_kinect_base_op" value="0" />
+	<property name="high_kinect_base_oy" value="0" />
 </robot>

File: elektron_description/urdf/tower/tower.urdf.xacro (robot description, xacro)
@@ -5,4 +5,17 @@
 <xacro:include filename="$(find elektron_description)/urdf/sensors/kinect.urdf.xacro"/>
   <xacro:macro name="elektron_tower" params="parent camera_type id">
+  <joint name="high_kinect_base_joint_${id}" type="fixed">
+      <origin xyz="${high_kinect_base_px} ${high_kinect_base_py} ${high_kinect_base_pz}" rpy="${high_kinect_base_or} ${high_kinect_base_op} ${high_kinect_base_oy}"/>
+      <parent link="${parent}"/>
+      <child link="high_kinect_base_${id}" />
+    </joint>
+    <link name="high_kinect_base_${id}">
+    	    	 <inertial>
+		     <origin xyz="0 0 0" rpy="0 0 0"/>
+		     <mass value="0.1"/>
+		     <inertia ixx="1"  ixy="0"  ixz="0" iyy="1" iyz="0" izz="1" />
+   		</inertial>
+	</link>
+<sensor_kinect parent="high_kinect_base_${id}" id="tower_top"/>
    <joint name="head_base_joint_${id}" type="fixed">
       <origin xyz="${head_base_px} ${head_base_py} ${head_base_pz}" rpy="${head_base_or} ${head_base_op} ${head_base_oy}"/>
