Commit message: add tower, not stable

File: elektron_description/robots/elektron_Laser_NoTower.urdf.xacro (robot description, xacro)
@@ -5,4 +5,5 @@
 	xmlns:interface="http://playerstage.sourceforge.net/gazebo/xmlschema/#interface">
 	<property name="M_PI" value="3.14159"/>
+	<property name="elektron_control_input" value="diff_drive_controller" />
 	<property name="base_size_x" value="0.38" />
 	<property name="base_size_y" value="0.28" />
@@ -11,4 +12,12 @@
 	<property name="wheel_length" value="0.02" />
 	<property name="caster_wheel_offset_y" value="0.1675" />
+	  	<!-- include calibrated params -->
+    <xacro:include filename="$(find elektron_description)/urdf/elektron_properties.urdf.xacro"/>
+	<!-- INCLUDE SICK LMX100 LASER -->
+	<include filename="$(find elektron_description)/urdf/sensors/sick_laser_lmx_100.urdf" />
+	<!-- INCLUDE KINECT -->
+	<include filename="$(find elektron_description)/urdf/sensors/kinect.urdf.xacro"/>
+	<!-- INCLUDE PID gazebo control -->
+	<include filename="$(find elektron_control)/gazebo/elektron_gazebo_control.urdf.xacro"/>
 	<!-- ROBOT BASE DEFINITION -->
 	<link name="base_link">
@@ -85,8 +94,18 @@
 		m="0"/>
 	<xacro:erratic_wheel suffix="right_rear" parent="base_link" reflect="-1" offset="-0.15"	m="0"/>
-	<!-- INCLUDE SICK LMX100 LASER -->
-	<include filename="$(find elektron_description)/urdf/sensors/sick_laser_lmx_100.urdf" />
-	<!-- add differentional drive to wheels -->
-	<gazebo>
+<!-- ADD KINECT -->
+    <joint name="bottom_kinect_joint" type="fixed">
+      <origin xyz="${kinect_px} ${kinect_py} ${kinect_pz}" rpy="${kinect_or} ${kinect_op} ${kinect_oy}"/>
+      <parent link="base_link"/>
+      <child link="bottom_kinect_link" />
+    </joint>
+    <link name="bottom_kinect_link"/>
+	<sensor_kinect parent="bottom_kinect_link" id="bottom"/>
+	<!-- SET gazebo-ROS CONTROL -->
+	<xacro:if value="${elektron_control_input == 'pid'}">
+		<elektron_PID_control_gazebo/>
+	</xacro:if>
+	<xacro:if value="${elektron_control_input == 'diff_drive_controller'}">
+		<gazebo>
 		<plugin name="differential_drive_controller" filename="libgazebo_ros_diff_drive.so">
 			<alwaysOn>true</alwaysOn>
@@ -103,51 +122,4 @@
 		</plugin>
 	</gazebo>
-	<!-- SET gazebo-ROS CONTROL -->
-	<gazebo>
-	  	<plugin name="gazebo_ros_control" filename="libgazebo_ros_control.so">
-	    	<robotNamespace>/elektron</robotNamespace>
-	  	</plugin>
-	</gazebo>
-	<!-- ADD position CONTROLLER - left wheel -->
-	<transmission name="tran_effort_left_wheel_joint">
-		<type>effort_controllers/JointPositionController</type>
-		<joint name="base_link_left_wheel_joint">
-			<hardwareInterface>EffortJointInterface</hardwareInterface>
-		</joint>
-		<actuator name="motor_base_link_left_wheel_joint">
-			<hardwareInterface>EffortJointInterface</hardwareInterface>
-			<mechanicalReduction>1</mechanicalReduction>
-		</actuator>
-	</transmission>
-	<!-- ADD position CONTROLLER - right wheel -->
-	<transmission name="tran_effort_right_wheel_joint">
-		<type>effort_controllers/JointPositionController</type>
-		<joint name="base_link_right_wheel_joint">
-			<hardwareInterface>EffortJointInterface</hardwareInterface>
-		</joint>
-		<actuator name="motor_base_link_right_wheel_joint">
-			<hardwareInterface>EffortJointInterface</hardwareInterface>
-      			<mechanicalReduction>1</mechanicalReduction>
-    		</actuator>
-  	</transmission>
-	<!-- ADD velocity CONTROLLER - left wheel -->
-  	<transmission name="tran_vel_left_wheel_joint">
-    		<type>effort_controllers/JointVelocityController</type>
-    		<joint name="base_link_left_wheel_joint">
-      			<hardwareInterface>VelocityJointInterface</hardwareInterface>
-    		</joint>
-    		<actuator name="motor_base_link_left_wheel_joint">
-      			<hardwareInterface>VelocityJointInterface</hardwareInterface>
-    		</actuator>
-  	</transmission>
-	<!-- ADD velocity CONTROLLER - right wheel -->
-	<transmission name="tran_vel_right_wheel_joint">
-		<type>effort_controllers/JointVelocityController</type>
-		<joint name="base_link_right_wheel_joint">
-     			<hardwareInterface>VelocityJointInterface</hardwareInterface>
-    		</joint>
-    		<actuator name="motor_base_link_right_wheel_joint">
-      			<hardwareInterface>VelocityJointInterface</hardwareInterface>
-    		</actuator>
-  	</transmission>
+	</xacro:if>
 </robot>

File: elektron_description/robots/elektron_NoLaser_NoTower.urdf.xacro (robot description, xacro)
@@ -5,4 +5,5 @@
 	xmlns:interface="http://playerstage.sourceforge.net/gazebo/xmlschema/#interface">
 	<property name="M_PI" value="3.14159"/>
+	<property name="elektron_control_input" value="diff_drive_controller" />
 	<property name="base_size_x" value="0.38" />
 	<property name="base_size_y" value="0.28" />
@@ -11,4 +12,10 @@
 	<property name="wheel_length" value="0.02" />
 	<property name="caster_wheel_offset_y" value="0.1675" />
+  	<!-- include calibrated params -->
+    <xacro:include filename="$(find elektron_description)/urdf/elektron_properties.urdf.xacro"/>
+	<!-- INCLUDE SICK LMX100 LASER -->
+	<!-- <include filename="$(find elektron_description)/urdf/sensors/sick_laser_lmx_100.urdf" />-->
+	<!-- INCLUDE KINECT -->
+	<include filename="$(find elektron_description)/urdf/sensors/kinect.urdf.xacro"/>
 	<!-- ROBOT BASE DEFINITION -->
 	<link name="base_link">
@@ -85,11 +92,18 @@
 		m="0"/>
 	<xacro:erratic_wheel suffix="right_rear" parent="base_link" reflect="-1" offset="-0.15"	m="0"/>
-	<!-- INCLUDE SICK LMX100 LASER -->
-	<!-- <include filename="$(find elektron_description)/urdf/sensors/sick_laser_lmx_100.urdf" />-->
-	<!-- INCLUDE KINECT -->
-	<include filename="$(find elektron_description)/urdf/sensors/kinect.urdf.xacro"/>
-	<sensor_kinect  parent="base_link"/>
-	<!-- add differentional drive to wheels -->
-	<gazebo>
+	<!-- ADD KINECT -->
+    <joint name="bottom_kinect_joint" type="fixed">
+      <origin xyz="${kinect_px} ${kinect_py} ${kinect_pz}" rpy="${kinect_or} ${kinect_op} ${kinect_oy}"/>
+      <parent link="base_link"/>
+      <child link="bottom_kinect_link" />
+    </joint>
+    <link name="bottom_kinect_link"/>
+	<sensor_kinect parent="bottom_kinect_link" id="bottom"/>
+	<!-- SET gazebo-ROS CONTROL -->
+	<xacro:if value="${elektron_control_input == 'pid'}">
+		<elektron_PID_control_gazebo/>
+	</xacro:if>
+	<xacro:if value="${elektron_control_input == 'diff_drive_controller'}">
+		<gazebo>
 		<plugin name="differential_drive_controller" filename="libgazebo_ros_diff_drive.so">
 			<alwaysOn>true</alwaysOn>
@@ -106,51 +120,4 @@
 		</plugin>
 	</gazebo>
-	<!-- SET gazebo-ROS CONTROL -->
-	<gazebo>
-	  	<plugin name="gazebo_ros_control" filename="libgazebo_ros_control.so">
-	    	<robotNamespace>/elektron</robotNamespace>
-	  	</plugin>
-	</gazebo>
-	<!-- ADD position CONTROLLER - left wheel -->
-	<transmission name="tran_effort_left_wheel_joint">
-		<type>effort_controllers/JointPositionController</type>
-		<joint name="base_link_left_wheel_joint">
-			<hardwareInterface>EffortJointInterface</hardwareInterface>
-		</joint>
-		<actuator name="motor_base_link_left_wheel_joint">
-			<hardwareInterface>EffortJointInterface</hardwareInterface>
-			<mechanicalReduction>1</mechanicalReduction>
-		</actuator>
-	</transmission>
-	<!-- ADD position CONTROLLER - right wheel -->
-	<transmission name="tran_effort_right_wheel_joint">
-		<type>effort_controllers/JointPositionController</type>
-		<joint name="base_link_right_wheel_joint">
-			<hardwareInterface>EffortJointInterface</hardwareInterface>
-		</joint>
-		<actuator name="motor_base_link_right_wheel_joint">
-			<hardwareInterface>EffortJointInterface</hardwareInterface>
-      			<mechanicalReduction>1</mechanicalReduction>
-    		</actuator>
-  	</transmission>
-	<!-- ADD velocity CONTROLLER - left wheel -->
-  	<transmission name="tran_vel_left_wheel_joint">
-    		<type>effort_controllers/JointVelocityController</type>
-    		<joint name="base_link_left_wheel_joint">
-      			<hardwareInterface>VelocityJointInterface</hardwareInterface>
-    		</joint>
-    		<actuator name="motor_base_link_left_wheel_joint">
-      			<hardwareInterface>VelocityJointInterface</hardwareInterface>
-    		</actuator>
-  	</transmission>
-	<!-- ADD velocity CONTROLLER - right wheel -->
-	<transmission name="tran_vel_right_wheel_joint">
-		<type>effort_controllers/JointVelocityController</type>
-		<joint name="base_link_right_wheel_joint">
-     			<hardwareInterface>VelocityJointInterface</hardwareInterface>
-    		</joint>
-    		<actuator name="motor_base_link_right_wheel_joint">
-      			<hardwareInterface>VelocityJointInterface</hardwareInterface>
-    		</actuator>
-  	</transmission>
+	</xacro:if>
 </robot>

File: elektron_description/urdf/elektron_properties.urdf.xacro (robot description, xacro)
@@ -19,9 +19,15 @@
      (currently in development and awaiting feedback)
    -->
-	<property name="kinect_px" value="0.15" />
+	<property name="kinect_px" value="0.1" />
 	<property name="kinect_py" value="0.0" />  <!-- Y varies for different configurations. get sets in sensors_urdf -->
-	<property name="kinect_pz" value="0.09"/>
+	<property name="kinect_pz" value="0.45"/>
 	<property name="kinect_or" value="0" />
 	<property name="kinect_op" value="0" />
 	<property name="kinect_oy" value="0" />
+  <property name="head_base_px" value="0.1" />
+  <property name="head_base_py" value="0.0" />  <!-- Y varies for different configurations. get sets in sensors_urdf -->
+  <property name="head_base_pz" value="0.75"/>
+  <property name="head_base_or" value="0" />
+  <property name="head_base_op" value="0" />
+  <property name="head_base_oy" value="0" />
 </robot>

File: elektron_description/urdf/sensors/kinect.urdf.xacro (robot description, xacro)
@@ -1,31 +1,30 @@
 <?xml version="1.0"?>
 <robot name="sensor_kinect" xmlns:xacro="http://ros.org/wiki/xacro">
-  <xacro:include filename="$(find elektron_description)/urdf/elektron_gazebo.urdf.xacro"/>
-  <xacro:include filename="$(find elektron_description)/urdf/elektron_properties.urdf.xacro"/>
+<xacro:include filename="$(find elektron_description)/urdf/elektron_gazebo.urdf.xacro"/>
   <xacro:property name="kinect_cam_py" value="-0.0125"/>
   <!-- Parameterised in part by the values in turtlebot_properties.urdf.xacro -->
-  <xacro:macro name="sensor_kinect" params="parent">
-    <joint name="camera_rgb_joint" type="fixed">
-      <origin xyz="${kinect_px} ${kinect_py} ${kinect_pz}" rpy="${kinect_or} ${kinect_op} ${kinect_oy}"/>
+  <xacro:macro name="sensor_kinect" params="parent id">
+    <joint name="kinect_camera_rgb_joint_${id}" type="fixed">
+      <origin xyz="0 0 0" rpy="0 0 0"/>
       <parent link="${parent}"/>
-      <child link="camera_rgb_frame" />
+      <child link="kinect_camera_rgb_frame_${id}" />
     </joint>
-    <link name="camera_rgb_frame"/>
-    <joint name="camera_rgb_optical_joint" type="fixed">
+    <link name="kinect_camera_rgb_frame_${id}"/>
+    <joint name="kinect_camera_rgb_optical_joint_${id}" type="fixed">
       <origin xyz="0 0 0" rpy="${-M_PI/2} 0 ${-M_PI/2}" />
-      <parent link="camera_rgb_frame" />
-      <child link="camera_rgb_optical_frame" />
+      <parent link="kinect_camera_rgb_frame_${id}" />
+      <child link="kinect_camera_rgb_optical_frame_${id}" />
     </joint>
-    <link name="camera_rgb_optical_frame"/>
-    <joint name="camera_joint" type="fixed">
+    <link name="kinect_camera_rgb_optical_frame_${id}"/>
+    <joint name="kinect_camera_joint_${id}" type="fixed">
       <origin xyz="-0.031 ${-kinect_cam_py} -0.016" rpy="0 0 0"/>
-      <parent link="camera_rgb_frame"/>
-      <child link="camera_link"/>
+      <parent link="kinect_camera_rgb_frame_${id}"/>
+      <child link="kinect_camera_link_${id}"/>
     </joint>
-      <link name="camera_link">
+      <link name="kinect_camera_link_${id}">
       <visual>
        <origin xyz="0 0 0" rpy="0 0 ${M_PI/2}"/>
         <geometry>
-         <mesh filename="package://elektron_description/meshes/sensors/kinect.dae"/>
+         <mesh filename="package://elektron_description/meshes/sensors/kinect/kinect.dae"/>
         </geometry>
       </visual>
@@ -47,18 +46,18 @@
          files. However, for Gazebo simulation we need them, so we add them here.
          (Hence, don't publish them additionally!) -->
-	<joint name="camera_depth_joint" type="fixed">
+	<joint name="kinect_camera_depth_joint_${id}" type="fixed">
 	  <origin xyz="0 ${2 * -kinect_cam_py} 0" rpy="0 0 0" />
-	  <parent link="camera_rgb_frame" />
-	  <child link="camera_depth_frame" />
+	  <parent link="kinect_camera_rgb_frame_${id}" />
+	  <child link="kinect_camera_depth_frame_${id}" />
 	</joint>
-	<link name="camera_depth_frame"/>
-	<joint name="camera_depth_optical_joint" type="fixed">
+	<link name="kinect_camera_depth_frame_${id}"/>
+	<joint name="kinect_camera_depth_optical_joint_${id}" type="fixed">
 	  <origin xyz="0 0 0" rpy="${-M_PI/2} 0 ${-M_PI/2}" />
-	  <parent link="camera_depth_frame" />
-	  <child link="camera_depth_optical_frame" />
+	  <parent link="kinect_camera_depth_frame_${id}" />
+	  <child link="kinect_camera_depth_optical_frame_${id}" />
 	</joint>
-	<link name="camera_depth_optical_frame"/>
+	<link name="kinect_camera_depth_optical_frame_${id}"/>
 	<!-- Kinect sensor for simulation -->
-	<turtlebot_sim_3dsensor/>
+	<elektron_sim_kinect id="${id}"/>
   </xacro:macro>
 </robot>

File: elektron_description/urdf/sensors/kinect_gazebo.urdf.xacro (robot description, xacro)
@@ -20,5 +20,5 @@
         </camera>
         <plugin name="kinect_camera_controller" filename="libgazebo_ros_openni_kinect.so">
-          <cameraName>camera</cameraName>
+          <cameraName>kinect</cameraName>
           <alwaysOn>true</alwaysOn>
           <updateRate>10</updateRate>
@@ -28,5 +28,5 @@
           <cameraInfoTopicName>rgb/camera_info</cameraInfoTopicName>
           <depthImageCameraInfoTopicName>depth/camera_info</depthImageCameraInfoTopicName>
-          <frameName>camera_depth_optical_frame</frameName>
+          <frameName>kinect_camera_depth_optical_frame</frameName>
           <baseline>0.1</baseline>
           <distortion_k1>0.0</distortion_k1>
