Commit message: all base configurations support, fixed ros_control support, fixed laser scans

File: elektron_description/robots/elektron_Laser_NoTower.urdf.xacro (robot description, xacro)
@@ -5,5 +5,5 @@
 	xmlns:interface="http://playerstage.sourceforge.net/gazebo/xmlschema/#interface">
 	<property name="M_PI" value="3.14159"/>
-	<property name="elektron_control_input" value="diff_drive_controller" />
+	<property name="elektron_control_input" value="pid" /> <!-- diff_drive_controller | pid -->
 	<property name="base_size_x" value="0.38" />
 	<property name="base_size_y" value="0.28" />
@@ -12,18 +12,21 @@
 	<property name="wheel_length" value="0.02" />
 	<property name="caster_wheel_offset_y" value="0.1675" />
-	  	<!-- include calibrated params -->
-    <xacro:include filename="$(find elektron_description)/urdf/elektron_properties.urdf.xacro"/>
-	<!-- INCLUDE SICK LMX100 LASER -->
+	<!-- INCLUDE SICK LMX100 LASER-->
 	<include filename="$(find elektron_description)/urdf/sensors/sick_laser_lmx_100.urdf" />
 	<!-- INCLUDE KINECT -->
 	<include filename="$(find elektron_description)/urdf/sensors/kinect.urdf.xacro"/>
-	<!-- INCLUDE PID gazebo control -->
+	<!-- INCLUDE TOWER
+	<include filename="$(find elektron_description)/urdf/tower/tower.urdf.xacro"/>-->
+  	<!-- include calibrated params -->
+    <xacro:include filename="$(find elektron_description)/urdf/elektron_properties.urdf.xacro"/>
+  	<!-- include gazebo control -->
 	<include filename="$(find elektron_control)/gazebo/elektron_gazebo_control.urdf.xacro"/>
+	<!-- <include filename="$(find elektron_control)/gazebo/tower_gazebo_control.urdf.xacro"/> -->
 	<!-- ROBOT BASE DEFINITION -->
 	<link name="base_link">
 		<inertial>
-			<mass value="15" />
+			<mass value="30" />
 			<origin xyz="-0.0 0 ${base_size_z/2}" />
-			<inertia ixx="1.0" ixy="0.0" ixz="0.0" iyy="1.0" iyz="0.0" izz="1.0" />
+			<inertia ixx="100.0" ixy="10.0" ixz="100.0" iyy="100.0" iyz="100.0" izz="100.0" />
 		</inertial>
 		<visual>
@@ -45,5 +48,5 @@
 	</link>
 	<!-- WHEELS MACRO -->
-	<xacro:macro name="erratic_wheel" params="suffix parent reflect offset m">
+	<xacro:macro name="erratic_wheel" params="suffix parent reflect offset m mimic">
 			<joint name="${parent}_${suffix}_wheel_joint" type="continuous">
 				<origin xyz="${offset} ${reflect*caster_wheel_offset_y} ${wheel_radius}" rpy="0	0 0"/>
@@ -55,4 +58,10 @@
 				<child link="${parent}_${suffix}_wheel_link" />
 	 			<dynamics damping="0.0" friction="0.0"/>
+	 			<xacro:if value="${mimic == 'left'}">
+		 			<mimic joint="${parent}_${mimic}_wheel_joint"/>
+				</xacro:if>
+	 			<xacro:if value="${mimic == 'right'}">
+		 			<mimic joint="${parent}_${mimic}_wheel_joint"/>
+				</xacro:if>
 			</joint>
 			<link name="${parent}_${suffix}_wheel_link">
@@ -87,11 +96,11 @@
 	</xacro:macro>
 	<!-- WHEELS DEFINITION -->
-	<xacro:erratic_wheel suffix="left" parent="base_link" reflect="1" offset="0" m="0.900"/>
-	<xacro:erratic_wheel suffix="left_front" parent="base_link" reflect="1" offset="0.15" m="0"/>
-	<xacro:erratic_wheel suffix="left_rear" parent="base_link" reflect="1" offset="-0.15" m="0"/>
-	<xacro:erratic_wheel suffix="right" parent="base_link" reflect="-1" offset="0" m="0.900"/>
+	<xacro:erratic_wheel suffix="left" parent="base_link" reflect="1" offset="0" m="0.900" mimic="none"/>
+	<xacro:erratic_wheel suffix="left_front" parent="base_link" reflect="1" offset="0.15" m="0" mimic="left"/>
+	<xacro:erratic_wheel suffix="left_rear" parent="base_link" reflect="1" offset="-0.15" m="0" mimic="left"/>
+	<xacro:erratic_wheel suffix="right" parent="base_link" reflect="-1" offset="0" m="0.900" mimic="none"/>
 	<xacro:erratic_wheel suffix="right_front" parent="base_link" reflect="-1" offset="0.15"
-		m="0"/>
-	<xacro:erratic_wheel suffix="right_rear" parent="base_link" reflect="-1" offset="-0.15"	m="0"/>
+		m="0" mimic="right"/>
+	<xacro:erratic_wheel suffix="right_rear" parent="base_link" reflect="-1" offset="-0.15"	m="0" mimic="right"/>
 <!-- ADD KINECT -->
     <joint name="bottom_kinect_joint" type="fixed">
@@ -102,4 +111,7 @@
     <link name="bottom_kinect_link"/>
 	<sensor_kinect parent="bottom_kinect_link" id="bottom"/>
+	<!-- ADD TOWER -->
+	<!-- <elektron_tower parent="base_link" camera_type="rgb_camera" id="1"/> camera_type avaliable: kinect | rgb_camera
+	<tower_PID_control_gazebo/>-->
 	<!-- SET gazebo-ROS CONTROL -->
 	<xacro:if value="${elektron_control_input == 'pid'}">

File: elektron_description/robots/elektron_Laser_Tower-kinect.urdf.xacro (robot description, xacro)
@@ -12,15 +12,15 @@
 	<property name="wheel_length" value="0.02" />
 	<property name="caster_wheel_offset_y" value="0.1675" />
-	<!-- INCLUDE SICK LMX100 LASER
-	<include filename="$(find elektron_description)/urdf/sensors/sick_laser_lmx_100.urdf" /> -->
+	<!-- INCLUDE SICK LMX100 LASER -->
+	<include filename="$(find elektron_description)/urdf/sensors/sick_laser_lmx_100.urdf" />
 	<!-- INCLUDE KINECT -->
 	<include filename="$(find elektron_description)/urdf/sensors/kinect.urdf.xacro"/>
-	<!-- INCLUDE TOWER
-	<include filename="$(find elektron_description)/urdf/tower/tower.urdf.xacro"/>-->
+	<!-- INCLUDE TOWER -->
+	<include filename="$(find elektron_description)/urdf/tower/tower.urdf.xacro"/>
   	<!-- include calibrated params -->
     <xacro:include filename="$(find elektron_description)/urdf/elektron_properties.urdf.xacro"/>
   	<!-- include gazebo control -->
 	<include filename="$(find elektron_control)/gazebo/elektron_gazebo_control.urdf.xacro"/>
-	<!-- <include filename="$(find elektron_control)/gazebo/tower_gazebo_control.urdf.xacro"/> -->
+	<include filename="$(find elektron_control)/gazebo/tower_gazebo_control.urdf.xacro"/>
 	<!-- ROBOT BASE DEFINITION -->
 	<link name="base_link">
@@ -112,6 +112,6 @@
 	<sensor_kinect parent="bottom_kinect_link" id="bottom"/>
 	<!-- ADD TOWER -->
-	<!-- <elektron_tower parent="base_link" camera_type="rgb_camera" id="1"/> camera_type avaliable: kinect | rgb_camera
-	<tower_PID_control_gazebo/>-->
+	<elektron_tower parent="base_link" camera_type="kinect" id="1"/> <!-- camera_type avaliable: kinect | rgb_camera -->
+	<tower_PID_control_gazebo/>
 	<!-- SET gazebo-ROS CONTROL -->
 	<xacro:if value="${elektron_control_input == 'pid'}">

File: elektron_description/robots/elektron_Laser_Tower-rgb.urdf.xacro (robot description, xacro)
@@ -12,15 +12,15 @@
 	<property name="wheel_length" value="0.02" />
 	<property name="caster_wheel_offset_y" value="0.1675" />
-	<!-- INCLUDE SICK LMX100 LASER
-	<include filename="$(find elektron_description)/urdf/sensors/sick_laser_lmx_100.urdf" /> -->
+	<!-- INCLUDE SICK LMX100 LASER -->
+	<include filename="$(find elektron_description)/urdf/sensors/sick_laser_lmx_100.urdf" />
 	<!-- INCLUDE KINECT -->
 	<include filename="$(find elektron_description)/urdf/sensors/kinect.urdf.xacro"/>
-	<!-- INCLUDE TOWER
-	<include filename="$(find elektron_description)/urdf/tower/tower.urdf.xacro"/>-->
+	<!-- INCLUDE TOWER -->
+	<include filename="$(find elektron_description)/urdf/tower/tower.urdf.xacro"/>
   	<!-- include calibrated params -->
     <xacro:include filename="$(find elektron_description)/urdf/elektron_properties.urdf.xacro"/>
   	<!-- include gazebo control -->
 	<include filename="$(find elektron_control)/gazebo/elektron_gazebo_control.urdf.xacro"/>
-	<!-- <include filename="$(find elektron_control)/gazebo/tower_gazebo_control.urdf.xacro"/> -->
+	<include filename="$(find elektron_control)/gazebo/tower_gazebo_control.urdf.xacro"/>
 	<!-- ROBOT BASE DEFINITION -->
 	<link name="base_link">
@@ -112,6 +112,6 @@
 	<sensor_kinect parent="bottom_kinect_link" id="bottom"/>
 	<!-- ADD TOWER -->
-	<!-- <elektron_tower parent="base_link" camera_type="rgb_camera" id="1"/> camera_type avaliable: kinect | rgb_camera
-	<tower_PID_control_gazebo/>-->
+	<elektron_tower parent="base_link" camera_type="rgb_camera" id="1"/> <!-- camera_type avaliable: kinect | rgb_camera -->
+	<tower_PID_control_gazebo/>
 	<!-- SET gazebo-ROS CONTROL -->
 	<xacro:if value="${elektron_control_input == 'pid'}">

File: elektron_description/robots/elektron_NoLaser_Tower-kinect.urdf.xacro (robot description, xacro)
@@ -16,11 +16,11 @@
 	<!-- INCLUDE KINECT -->
 	<include filename="$(find elektron_description)/urdf/sensors/kinect.urdf.xacro"/>
-	<!-- INCLUDE TOWER
-	<include filename="$(find elektron_description)/urdf/tower/tower.urdf.xacro"/>-->
+	<!-- INCLUDE TOWER -->
+	<include filename="$(find elektron_description)/urdf/tower/tower.urdf.xacro"/>
   	<!-- include calibrated params -->
     <xacro:include filename="$(find elektron_description)/urdf/elektron_properties.urdf.xacro"/>
   	<!-- include gazebo control -->
 	<include filename="$(find elektron_control)/gazebo/elektron_gazebo_control.urdf.xacro"/>
-	<!-- <include filename="$(find elektron_control)/gazebo/tower_gazebo_control.urdf.xacro"/> -->
+	<include filename="$(find elektron_control)/gazebo/tower_gazebo_control.urdf.xacro"/>
 	<!-- ROBOT BASE DEFINITION -->
 	<link name="base_link">
@@ -112,6 +112,6 @@
 	<sensor_kinect parent="bottom_kinect_link" id="bottom"/>
 	<!-- ADD TOWER -->
-	<!-- <elektron_tower parent="base_link" camera_type="rgb_camera" id="1"/> camera_type avaliable: kinect | rgb_camera
-	<tower_PID_control_gazebo/>-->
+	<elektron_tower parent="base_link" camera_type="kinect" id="1"/> <!-- camera_type avaliable: kinect | rgb_camera -->
+	<tower_PID_control_gazebo/>
 	<!-- SET gazebo-ROS CONTROL -->
 	<xacro:if value="${elektron_control_input == 'pid'}">

File: elektron_description/robots/elektron_NoLaser_Tower-rgb.urdf.xacro (robot description, xacro)
@@ -16,11 +16,11 @@
 	<!-- INCLUDE KINECT -->
 	<include filename="$(find elektron_description)/urdf/sensors/kinect.urdf.xacro"/>
-	<!-- INCLUDE TOWER
-	<include filename="$(find elektron_description)/urdf/tower/tower.urdf.xacro"/>-->
+	<!-- INCLUDE TOWER -->
+	<include filename="$(find elektron_description)/urdf/tower/tower.urdf.xacro"/>
   	<!-- include calibrated params -->
     <xacro:include filename="$(find elektron_description)/urdf/elektron_properties.urdf.xacro"/>
   	<!-- include gazebo control -->
 	<include filename="$(find elektron_control)/gazebo/elektron_gazebo_control.urdf.xacro"/>
-	<!-- <include filename="$(find elektron_control)/gazebo/tower_gazebo_control.urdf.xacro"/> -->
+	<include filename="$(find elektron_control)/gazebo/tower_gazebo_control.urdf.xacro"/>
 	<!-- ROBOT BASE DEFINITION -->
 	<link name="base_link">
@@ -112,6 +112,6 @@
 	<sensor_kinect parent="bottom_kinect_link" id="bottom"/>
 	<!-- ADD TOWER -->
-	<!-- <elektron_tower parent="base_link" camera_type="rgb_camera" id="1"/> camera_type avaliable: kinect | rgb_camera
-	<tower_PID_control_gazebo/>-->
+	<elektron_tower parent="base_link" camera_type="rgb_camera" id="1"/> <!-- camera_type avaliable: kinect | rgb_camera -->
+	<tower_PID_control_gazebo/>
 	<!-- SET gazebo-ROS CONTROL -->
 	<xacro:if value="${elektron_control_input == 'pid'}">

File: elektron_description/urdf/elektron_gazebo.urdf.xacro (robot description, xacro)
@@ -2,6 +2,6 @@
 <robot name="elektron_gazebo" xmlns:xacro="http://ros.org/wiki/xacro">
   <!-- Microsoft Kinect / ASUS Xtion PRO Live for simulation -->
-  <xacro:macro name="elektron_sim_kinect" params="id">
-    <gazebo reference="kinect_camera_link_${id}">
+  <xacro:macro name="elektron_sim_kinect" params="id reference">
+    <gazebo reference="${reference}">
       <sensor type="depth" name="kinect_camera_${id}">
         <always_on>true</always_on>
@@ -41,9 +41,9 @@
   </xacro:macro>
   <!-- head camera -->
-  <xacro:macro name="elektron_sim_cam_head">
-  <gazebo reference="camera_head_link">
-    <sensor type="camera" name="camera1">
+  <xacro:macro name="elektron_sim_cam_head" params="id reference frame">
+  <gazebo reference="${reference}">
+    <sensor type="camera" name="camera_${id}">
       <update_rate>30.0</update_rate>
-      <camera name="head">
+      <camera name="camera_${id}">
         <horizontal_fov>1.3962634</horizontal_fov>
         <image>
@@ -65,11 +65,11 @@
         </noise>
       </camera>
-      <plugin name="camera_controller" filename="libgazebo_ros_camera.so">
+      <plugin name="camera_controller_${id}" filename="libgazebo_ros_camera.so">
         <alwaysOn>true</alwaysOn>
         <updateRate>0.0</updateRate>
-        <cameraName>elektron/camera_head</cameraName>
-        <imageTopicName>camera_head/image_raw</imageTopicName>
-        <cameraInfoTopicName>camera_head/camera_info</cameraInfoTopicName>
-        <frameName>camera_link</frameName>
+        <cameraName>elektron/camera_${id}</cameraName>
+        <imageTopicName>/image_raw</imageTopicName>
+        <cameraInfoTopicName>/camera_info</cameraInfoTopicName>
+        <frameName>${frame}</frameName>
         <hackBaseline>0.07</hackBaseline>
         <distortionK1>0.0</distortionK1>

File: elektron_description/urdf/elektron_properties.urdf.xacro (robot description, xacro)
@@ -26,5 +26,5 @@
 	<property name="kinect_oy" value="0" />
   <property name="head_base_px" value="0.1" />
-  <property name="head_base_py" value="0.0" />  <!-- Y varies for different configurations. get sets in sensors_urdf -->
+  <property name="head_base_py" value="0.0" />
   <property name="head_base_pz" value="0.75"/>
   <property name="head_base_or" value="0" />

File: elektron_description/urdf/sensors/kinect.urdf.xacro (robot description, xacro)
@@ -6,5 +6,5 @@
   <xacro:macro name="sensor_kinect" params="parent id">
     <joint name="kinect_camera_rgb_joint_${id}" type="fixed">
-      <origin xyz="0 0 0" rpy="0 0 0"/>
+      <origin xyz="0.06 0 0.05" rpy="0 0 0"/>
       <parent link="${parent}"/>
       <child link="kinect_camera_rgb_frame_${id}" />
@@ -59,5 +59,5 @@
 	<link name="kinect_camera_depth_optical_frame_${id}"/>
 	<!-- Kinect sensor for simulation -->
-	<elektron_sim_kinect id="${id}"/>
+	<elektron_sim_kinect id="${id}" reference="kinect_camera_link_${id}"/>
   </xacro:macro>
 </robot>

File: elektron_description/urdf/sensors/rgb_camera.urdf.xacro (robot description, xacro)
@@ -2,23 +2,23 @@
 <robot name="elektron_rgb_camera" xmlns:xacro="http://ros.org/wiki/xacro">
 <xacro:include filename="$(find elektron_description)/urdf/elektron_gazebo.urdf.xacro"/>
-  <xacro:macro name="elektron_rgb_camera" params="parent">
-    <joint name="head_camera_joint" type="fixed">
-      <origin xyz="-0.05 0.0 0.05" rpy="0 0 0"/>
+  <xacro:macro name="elektron_rgb_camera" params="parent id">
+    <joint name="camera_joint_${id}" type="fixed">
+      <origin xyz="0.0 0.0 0" rpy="0 0 0"/>
       <parent link="${parent}"/>
-      <child link="head_camera_link"/>
+      <child link="camera_link_${id}"/>
     </joint>
-      <link name="head_camera_link">
+      <link name="camera_link_${id}">
       <visual>
        <origin xyz="0 0 0" rpy="0 0 ${M_PI/2}"/>
         <geometry>
-         <mesh filename="package://elektron_description/meshes/sensors/head_camera/head_camera.dae"/>
+         <mesh filename="package://elektron_description/meshes/sensors/head_camera/scaled_camera.dae"/>
         </geometry>
       </visual>
-  	  <collision>
+      <collision>
         <origin xyz="0.0 0.0 0.0" rpy="0 0 0"/>
-  	    <geometry>
-  	      <box size="0.07271 0.27794 0.073"/>
-  	    </geometry>
-  	  </collision>
+        <geometry>
+          <box size="0.07271 0.27794 0.073"/>
+        </geometry>
+      </collision>
       <inertial>
         <mass value="0.564" />
@@ -29,5 +29,19 @@
       </inertial>
     </link>
-      <elektron_sim_cam_head/>
+        <joint name="camera_optical_joint_${id}" type="fixed">
+      <origin xyz="0.05 0.0 0.04" rpy="0 0 0"/>
+      <parent link="camera_link_${id}"/>
+      <child link="camera_optical_link_${id}"/>
+    </joint>
+      <link name="camera_optical_link_${id}">
+        <inertial>
+        <mass value="0.01" />
+        <origin xyz="0 0 0" />
+        <inertia ixx="0.003881243" ixy="0.0" ixz="0.0"
+                 iyy="0.000498940" iyz="0.0"
+                 izz="0.003879257" />
+      </inertial>
+    </link>
+      <elektron_sim_cam_head reference="camera_optical_link_${id}" id="${id}" frame="camera_optical_link_${id}"/>
       </xacro:macro>
 </robot>

File: elektron_description/urdf/tower/tower.urdf.xacro (robot description, xacro)
@@ -4,44 +4,74 @@
 <xacro:include filename="$(find elektron_description)/urdf/sensors/rgb_camera.urdf.xacro"/>
 <xacro:include filename="$(find elektron_description)/urdf/sensors/kinect.urdf.xacro"/>
-  <xacro:macro name="elektron_tower" params="parent camera_type">
-   <joint name="head_base_joint" type="fixed">
+  <xacro:macro name="elektron_tower" params="parent camera_type id">
+   <joint name="head_base_joint_${id}" type="fixed">
       <origin xyz="${head_base_px} ${head_base_py} ${head_base_pz}" rpy="${head_base_or} ${head_base_op} ${head_base_oy}"/>
       <parent link="${parent}"/>
       <child link="head_base" />
     </joint>
-    <link name="head_base"/>
-    <joint name="head_yaw_revolute_joint" type="revolute">
+    <link name="head_base">
+    	    	 <inertial>
+		     <origin xyz="0 0 0" rpy="0 0 0"/>
+		     <mass value="0.1"/>
+		     <inertia ixx="1"  ixy="0"  ixz="0" iyy="1" iyz="0" izz="1" />
+   		</inertial>
+	</link>
+    <joint name="head_yaw_revolute_joint_${id}" type="revolute">
       <origin xyz="0 0 0" rpy="0 0 0" />
      <!-- --> <axis xyz="0 0 1"/>
       <limit effort="1000.0" lower="-${M_PI/2}" upper="${M_PI/2}" velocity="0.5"/>
       <parent link="head_base" />
-      <child link="head_bottom_revolute_link" />
+      <child link="head_bottom_revolute_link_${id}" />
     </joint>
-    <link name="head_bottom_revolute_link"/>
-    <joint name="head_yaw_fixed_joint" type="fixed">
+    <link name="head_bottom_revolute_link_${id}">
+    	 <inertial>
+		     <origin xyz="0 0 0" rpy="0 0 0"/>
+		     <mass value="0.1"/>
+		     <inertia ixx="1"  ixy="0"  ixz="0" iyy="0" iyz="0" izz="1" />
+   		</inertial>
+	</link>
+    <joint name="head_yaw_fixed_joint_${id}" type="fixed">
       <origin xyz="0 0 0" rpy="0 0 0" />
-      <parent link="head_bottom_revolute_link" />
-      <child link="head_bottom_fixed_link" />
+      <parent link="head_bottom_revolute_link_${id}" />
+      <child link="head_bottom_fixed_link_${id}" />
     </joint>
-    <link name="head_bottom_fixed_link"/>
-    <joint name="head_pitch_revolute_joint" type="revolute">
+    <link name="head_bottom_fixed_link_${id}">
+    	<inertial>
+		     <origin xyz="0 0 0" rpy="0 0 0"/>
+		     <mass value="0.1"/>
+		     <inertia ixx="1"  ixy="0"  ixz="0" iyy="1" iyz="0" izz="1" />
+   		</inertial>
+	</link>
+    <joint name="head_pitch_revolute_joint_${id}" type="revolute">
       <origin xyz="0 0 0.05" rpy="0 0 0" />
       <axis xyz="0 1 0"/>
       <limit effort="1000.0" lower="-${M_PI/2}" upper="${M_PI/2}" velocity="0.5"/>
-      <parent link="head_bottom_fixed_link" />
-      <child link="head_upper_revolute_link" />
+      <parent link="head_bottom_fixed_link_${id}" />
+      <child link="head_upper_revolute_link_${id}" />
     </joint>
-    <link name="head_upper_revolute_link"/>
-    <joint name="head_pitch_fixed_joint" type="fixed">
-      <origin xyz="0 0 0.05" rpy="0 0 0" />
-      <parent link="head_upper_revolute_link" />
-      <child link="head_upper_fixed_link" />
+    <link name="head_upper_revolute_link_${id}">
+    	<inertial>
+		     <origin xyz="0 0 0" rpy="0 0 0"/>
+		     <mass value="0.1"/>
+		     <inertia ixx="1"  ixy="0"  ixz="0" iyy="1" iyz="0" izz="1" />
+   		</inertial>
+	</link>
+    <joint name="head_pitch_fixed_joint_${id}" type="fixed">
+      <origin xyz="0.05 0 0.05" rpy="0 0 0" />
+      <parent link="head_upper_revolute_link_${id}" />
+      <child link="head_upper_fixed_link_${id}" />
     </joint>
-    <link name="head_upper_fixed_link"/>
+    <link name="head_upper_fixed_link_${id}">
+    	<inertial>
+		     <origin xyz="0 0 0" rpy="0 0 0"/>
+		     <mass value="0.1"/>
+		     <inertia ixx="1"  ixy="0"  ixz="0" iyy="1" iyz="0" izz="1" />
+   		</inertial>
+	</link>
 	<xacro:if value="${camera_type == 'kinect'}">
-		<sensor_kinect parent="head_upper_fixed_link" id="head"/>
+		<sensor_kinect parent="head_upper_fixed_link_${id}" id="head"/>
 	</xacro:if>
 	<xacro:if value="${camera_type == 'rgb_camera'}">
-		<elektron_rgb_camera parent="head_upper_fixed_link"/>
+		<elektron_rgb_camera parent="head_upper_fixed_link_${id}" id="head"/>
 	</xacro:if>
  <!--   <joint name="head_camera_joint" type="fixed">
