Commit message: compatibility with ros-indigo, add package.xml dependencies, move sick mesh to meshes folder

File: elektron_description/robots/elektron_Laser_NoTower.urdf.xacro (robot description, xacro)
@@ -12,15 +12,15 @@
 	<property name="wheel_length" value="0.02" />
 	<property name="caster_wheel_offset_y" value="0.1675" />
-	<!-- INCLUDE SICK LMX100 LASER-->
-	<include filename="$(find elektron_description)/urdf/sensors/sick_laser_lmx_100.urdf" />
+	<!-- INCLUDE SICK LMX100 LASER -->
+	<xacro:include filename="$(find elektron_description)/urdf/sensors/sick_laser_lmx_100.urdf" />
 	<!-- INCLUDE KINECT -->
-	<include filename="$(find elektron_description)/urdf/sensors/kinect.urdf.xacro"/>
+	<xacro:include filename="$(find elektron_description)/urdf/sensors/kinect.urdf.xacro"/>
 	<!-- INCLUDE TOWER
-	<include filename="$(find elektron_description)/urdf/tower/tower.urdf.xacro"/>-->
+	<xacro:include filename="$(find elektron_description)/urdf/tower/tower.urdf.xacro"/>-->
   	<!-- include calibrated params -->
     <xacro:include filename="$(find elektron_description)/urdf/elektron_properties.urdf.xacro"/>
   	<!-- include gazebo control -->
-	<include filename="$(find elektron_control)/gazebo/elektron_gazebo_control.urdf.xacro"/>
-	<!-- <include filename="$(find elektron_control)/gazebo/tower_gazebo_control.urdf.xacro"/> -->
+	<xacro:include filename="$(find elektron_control)/gazebo/elektron_gazebo_control.urdf.xacro"/>
+	<!-- <xacro:include filename="$(find elektron_control)/gazebo/tower_gazebo_control.urdf.xacro"/> -->
 	<!-- ROBOT BASE DEFINITION -->
 	<link name="base_link">

File: elektron_description/robots/elektron_Laser_Tower-kinect.urdf.xacro (robot description, xacro)
@@ -5,5 +5,5 @@
 	xmlns:interface="http://playerstage.sourceforge.net/gazebo/xmlschema/#interface">
 	<property name="M_PI" value="3.14159"/>
-	<property name="elektron_control_input" value="pid" /> <!-- diff_drive_controller | pid -->
+	<property name="elektron_control_input" value="1" /> <!-- 0 = diff_drive_controller | 1 = pid -->
 	<property name="base_size_x" value="0.38" />
 	<property name="base_size_y" value="0.28" />
@@ -13,14 +13,14 @@
 	<property name="caster_wheel_offset_y" value="0.1675" />
 	<!-- INCLUDE SICK LMX100 LASER -->
-	<include filename="$(find elektron_description)/urdf/sensors/sick_laser_lmx_100.urdf" />
+	<xacro:include filename="$(find elektron_description)/urdf/sensors/sick_laser_lmx_100.urdf" />
 	<!-- INCLUDE KINECT -->
-	<include filename="$(find elektron_description)/urdf/sensors/kinect.urdf.xacro"/>
+	<xacro:include filename="$(find elektron_description)/urdf/sensors/kinect.urdf.xacro"/>
 	<!-- INCLUDE TOWER -->
-	<include filename="$(find elektron_description)/urdf/tower/tower.urdf.xacro"/>
+	<xacro:include filename="$(find elektron_description)/urdf/tower/tower.urdf.xacro"/>
   	<!-- include calibrated params -->
     <xacro:include filename="$(find elektron_description)/urdf/elektron_properties.urdf.xacro"/>
   	<!-- include gazebo control -->
-	<include filename="$(find elektron_control)/gazebo/elektron_gazebo_control.urdf.xacro"/>
-	<include filename="$(find elektron_control)/gazebo/tower_gazebo_control.urdf.xacro"/>
+	<xacro:include filename="$(find elektron_control)/gazebo/elektron_gazebo_control.urdf.xacro"/>
+	<xacro:include filename="$(find elektron_control)/gazebo/tower_gazebo_control.urdf.xacro"/>
 	<!-- ROBOT BASE DEFINITION -->
 	<link name="base_link">
@@ -48,5 +48,5 @@
 	</link>
 	<!-- WHEELS MACRO -->
-	<xacro:macro name="erratic_wheel" params="suffix parent reflect offset m mimic">
+	<xacro:macro name="erratic_wheel" params="suffix parent reflect offset m mimic mimic_wheel">
 			<joint name="${parent}_${suffix}_wheel_joint" type="continuous">
 				<origin xyz="${offset} ${reflect*caster_wheel_offset_y} ${wheel_radius}" rpy="0	0 0"/>
@@ -58,9 +58,6 @@
 				<child link="${parent}_${suffix}_wheel_link" />
 	 			<dynamics damping="0.0" friction="0.0"/>
-	 			<xacro:if value="${mimic == 'left'}">
-		 			<mimic joint="${parent}_${mimic}_wheel_joint"/>
-				</xacro:if>
-	 			<xacro:if value="${mimic == 'right'}">
-		 			<mimic joint="${parent}_${mimic}_wheel_joint"/>
+	 			<xacro:if value="${mimic}">
+		 			<mimic joint="${parent}_${mimic_wheel}_wheel_joint"/>
 				</xacro:if>
 			</joint>
@@ -96,11 +93,11 @@
 	</xacro:macro>
 	<!-- WHEELS DEFINITION -->
-	<xacro:erratic_wheel suffix="left" parent="base_link" reflect="1" offset="0" m="0.900" mimic="none"/>
-	<xacro:erratic_wheel suffix="left_front" parent="base_link" reflect="1" offset="0.15" m="0" mimic="left"/>
-	<xacro:erratic_wheel suffix="left_rear" parent="base_link" reflect="1" offset="-0.15" m="0" mimic="left"/>
-	<xacro:erratic_wheel suffix="right" parent="base_link" reflect="-1" offset="0" m="0.900" mimic="none"/>
+	<xacro:erratic_wheel suffix="left" parent="base_link" reflect="1" offset="0" m="0.900" mimic="0" mimic_wheel="left"/>
+	<xacro:erratic_wheel suffix="left_front" parent="base_link" reflect="1" offset="0.15" m="0" mimic="1" mimic_wheel="left"/>
+	<xacro:erratic_wheel suffix="left_rear" parent="base_link" reflect="1" offset="-0.15" m="0" mimic="1" mimic_wheel="left"/>
+	<xacro:erratic_wheel suffix="right" parent="base_link" reflect="-1" offset="0" m="0.900" mimic="0" mimic_wheel="left"/>
 	<xacro:erratic_wheel suffix="right_front" parent="base_link" reflect="-1" offset="0.15"
-		m="0" mimic="right"/>
-	<xacro:erratic_wheel suffix="right_rear" parent="base_link" reflect="-1" offset="-0.15"	m="0" mimic="right"/>
+		m="0" mimic="1" mimic_wheel="right" />
+	<xacro:erratic_wheel suffix="right_rear" parent="base_link" reflect="-1" offset="-0.15"	m="0" mimic="1" mimic_wheel="right"/>
 <!-- ADD KINECT -->
     <joint name="bottom_kinect_joint" type="fixed">
@@ -112,11 +109,11 @@
 	<sensor_kinect parent="bottom_kinect_link" id="bottom"/>
 	<!-- ADD TOWER -->
-	<elektron_tower parent="base_link" camera_type="kinect" id="1"/> <!-- camera_type avaliable: kinect | rgb_camera -->
+	<elektron_tower parent="base_link" camera_type="1" id="1"/> <!-- camera_type avaliable: 1 = kinect | 0 = rgb_camera -->
 	<tower_PID_control_gazebo/>
 	<!-- SET gazebo-ROS CONTROL -->
-	<xacro:if value="${elektron_control_input == 'pid'}">
+	<xacro:if value="${elektron_control_input}">
 		<elektron_PID_control_gazebo/>
 	</xacro:if>
-	<xacro:if value="${elektron_control_input == 'diff_drive_controller'}">
+	<xacro:unless value="${elektron_control_input}">
 		<gazebo>
 		<plugin name="differential_drive_controller" filename="libgazebo_ros_diff_drive.so">
@@ -134,4 +131,4 @@
 		</plugin>
 	</gazebo>
-	</xacro:if>
+	</xacro:unless>
 </robot>

File: elektron_description/robots/elektron_Laser_Tower-rgb.urdf.xacro (robot description, xacro)
@@ -13,14 +13,14 @@
 	<property name="caster_wheel_offset_y" value="0.1675" />
 	<!-- INCLUDE SICK LMX100 LASER -->
-	<include filename="$(find elektron_description)/urdf/sensors/sick_laser_lmx_100.urdf" />
+	<xacro:include filename="$(find elektron_description)/urdf/sensors/sick_laser_lmx_100.urdf" />
 	<!-- INCLUDE KINECT -->
-	<include filename="$(find elektron_description)/urdf/sensors/kinect.urdf.xacro"/>
+	<xacro:include filename="$(find elektron_description)/urdf/sensors/kinect.urdf.xacro"/>
 	<!-- INCLUDE TOWER -->
-	<include filename="$(find elektron_description)/urdf/tower/tower.urdf.xacro"/>
+	<xacro:include filename="$(find elektron_description)/urdf/tower/tower.urdf.xacro"/>
   	<!-- include calibrated params -->
     <xacro:include filename="$(find elektron_description)/urdf/elektron_properties.urdf.xacro"/>
   	<!-- include gazebo control -->
-	<include filename="$(find elektron_control)/gazebo/elektron_gazebo_control.urdf.xacro"/>
-	<include filename="$(find elektron_control)/gazebo/tower_gazebo_control.urdf.xacro"/>
+	<xacro:include filename="$(find elektron_control)/gazebo/elektron_gazebo_control.urdf.xacro"/>
+	<xacro:include filename="$(find elektron_control)/gazebo/tower_gazebo_control.urdf.xacro"/>
 	<!-- ROBOT BASE DEFINITION -->
 	<link name="base_link">

File: elektron_description/robots/elektron_NoLaser_NoTower.urdf.xacro (robot description, xacro)
@@ -13,14 +13,14 @@
 	<property name="caster_wheel_offset_y" value="0.1675" />
 	<!-- INCLUDE SICK LMX100 LASER
-	<include filename="$(find elektron_description)/urdf/sensors/sick_laser_lmx_100.urdf" /> -->
+	<xacro:include filename="$(find elektron_description)/urdf/sensors/sick_laser_lmx_100.urdf" /> -->
 	<!-- INCLUDE KINECT -->
-	<include filename="$(find elektron_description)/urdf/sensors/kinect.urdf.xacro"/>
+	<xacro:include filename="$(find elektron_description)/urdf/sensors/kinect.urdf.xacro"/>
 	<!-- INCLUDE TOWER
-	<include filename="$(find elektron_description)/urdf/tower/tower.urdf.xacro"/>-->
+	<xacro:include filename="$(find elektron_description)/urdf/tower/tower.urdf.xacro"/>-->
   	<!-- include calibrated params -->
     <xacro:include filename="$(find elektron_description)/urdf/elektron_properties.urdf.xacro"/>
   	<!-- include gazebo control -->
-	<include filename="$(find elektron_control)/gazebo/elektron_gazebo_control.urdf.xacro"/>
-	<!-- <include filename="$(find elektron_control)/gazebo/tower_gazebo_control.urdf.xacro"/> -->
+	<xacro:include filename="$(find elektron_control)/gazebo/elektron_gazebo_control.urdf.xacro"/>
+	<!-- <xacro:include filename="$(find elektron_control)/gazebo/tower_gazebo_control.urdf.xacro"/> -->
 	<!-- ROBOT BASE DEFINITION -->
 	<link name="base_link">

File: elektron_description/robots/elektron_NoLaser_Tower-kinect.urdf.xacro (robot description, xacro)
@@ -13,14 +13,14 @@
 	<property name="caster_wheel_offset_y" value="0.1675" />
 	<!-- INCLUDE SICK LMX100 LASER
-	<include filename="$(find elektron_description)/urdf/sensors/sick_laser_lmx_100.urdf" /> -->
+	<xacro:include filename="$(find elektron_description)/urdf/sensors/sick_laser_lmx_100.urdf" /> -->
 	<!-- INCLUDE KINECT -->
-	<include filename="$(find elektron_description)/urdf/sensors/kinect.urdf.xacro"/>
+	<xacro:include filename="$(find elektron_description)/urdf/sensors/kinect.urdf.xacro"/>
 	<!-- INCLUDE TOWER -->
-	<include filename="$(find elektron_description)/urdf/tower/tower.urdf.xacro"/>
+	<xacro:include filename="$(find elektron_description)/urdf/tower/tower.urdf.xacro"/>
   	<!-- include calibrated params -->
     <xacro:include filename="$(find elektron_description)/urdf/elektron_properties.urdf.xacro"/>
   	<!-- include gazebo control -->
-	<include filename="$(find elektron_control)/gazebo/elektron_gazebo_control.urdf.xacro"/>
-	<include filename="$(find elektron_control)/gazebo/tower_gazebo_control.urdf.xacro"/>
+	<xacro:include filename="$(find elektron_control)/gazebo/elektron_gazebo_control.urdf.xacro"/>
+	<xacro:include filename="$(find elektron_control)/gazebo/tower_gazebo_control.urdf.xacro"/>
 	<!-- ROBOT BASE DEFINITION -->
 	<link name="base_link">

File: elektron_description/robots/elektron_NoLaser_Tower-rgb.urdf.xacro (robot description, xacro)
@@ -13,14 +13,14 @@
 	<property name="caster_wheel_offset_y" value="0.1675" />
 	<!-- INCLUDE SICK LMX100 LASER
-	<include filename="$(find elektron_description)/urdf/sensors/sick_laser_lmx_100.urdf" /> -->
+	<xacro:include filename="$(find elektron_description)/urdf/sensors/sick_laser_lmx_100.urdf" /> -->
 	<!-- INCLUDE KINECT -->
-	<include filename="$(find elektron_description)/urdf/sensors/kinect.urdf.xacro"/>
+	<xacro:include filename="$(find elektron_description)/urdf/sensors/kinect.urdf.xacro"/>
 	<!-- INCLUDE TOWER -->
-	<include filename="$(find elektron_description)/urdf/tower/tower.urdf.xacro"/>
+	<xacro:include filename="$(find elektron_description)/urdf/tower/tower.urdf.xacro"/>
   	<!-- include calibrated params -->
     <xacro:include filename="$(find elektron_description)/urdf/elektron_properties.urdf.xacro"/>
   	<!-- include gazebo control -->
-	<include filename="$(find elektron_control)/gazebo/elektron_gazebo_control.urdf.xacro"/>
-	<include filename="$(find elektron_control)/gazebo/tower_gazebo_control.urdf.xacro"/>
+	<xacro:include filename="$(find elektron_control)/gazebo/elektron_gazebo_control.urdf.xacro"/>
+	<xacro:include filename="$(find elektron_control)/gazebo/tower_gazebo_control.urdf.xacro"/>
 	<!-- ROBOT BASE DEFINITION -->
 	<link name="base_link">

File: elektron_description/urdf/sensors/sick_laser_lmx_100.urdf (robot description, URDF)
Before this commit: robot None, 1 links, 1 joints
Links:
- link base_laser_link: geometry collision cylinder length=.05 radius=.05; visual mesh filename=package://elektron_description/meshes/sensors/laser/sick_lm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

File: elektron_description/urdf/tower/tower.urdf.xacro (robot description, xacro)
@@ -69,10 +69,10 @@
    		</inertial>
 	</link>
-	<xacro:if value="${camera_type == 'kinect'}">
+	<xacro:if value="${camera_type}">
 		<sensor_kinect parent="head_upper_fixed_link_${id}" id="head"/>
 	</xacro:if>
-	<xacro:if value="${camera_type == 'rgb_camera'}">
+	<xacro:unless value="${camera_type}">
 		<elektron_rgb_camera parent="head_upper_fixed_link_${id}" id="head"/>
-	</xacro:if>
+	</xacro:unless>
  <!--   <joint name="head_camera_joint" type="fixed">
       <origin xyz="-0.05 0.0 0.05" rpy="0 0 0"/>

Commit message: move elektron base mesh

File: elektron_description/robots/elektron_Laser_NoTower.urdf.xacro (robot description, xacro)
@@ -34,5 +34,5 @@
 			<geometry>
 				<!--<box size="0.38 0.28 0.20" />-->
-				<mesh filename="package://elektron_description/meshes/elektron_body.dae"/>
+				<mesh filename="package://elektron_description/meshes/base/elektron_body.dae"/>
 			</geometry>
 		</visual>

File: elektron_description/robots/elektron_Laser_Tower-kinect.urdf.xacro (robot description, xacro)
@@ -34,5 +34,5 @@
 			<geometry>
 				<!--<box size="0.38 0.28 0.20" />-->
-				<mesh filename="package://elektron_description/meshes/elektron_body.dae"/>
+				<mesh filename="package://elektron_description/meshes/base/elektron_body.dae"/>
 			</geometry>
 		</visual>

File: elektron_description/robots/elektron_Laser_Tower-rgb.urdf.xacro (robot description, xacro)
@@ -34,5 +34,5 @@
 			<geometry>
 				<!--<box size="0.38 0.28 0.20" />-->
-				<mesh filename="package://elektron_description/meshes/elektron_body.dae"/>
+				<mesh filename="package://elektron_description/meshes/base/elektron_body.dae"/>
 			</geometry>
 		</visual>

File: elektron_description/robots/elektron_NoLaser_NoTower.urdf.xacro (robot description, xacro)
@@ -34,5 +34,5 @@
 			<geometry>
 				<!--<box size="0.38 0.28 0.20" />-->
-				<mesh filename="package://elektron_description/meshes/elektron_body.dae"/>
+				<mesh filename="package://elektron_description/meshes/base/elektron_body.dae"/>
 			</geometry>
 		</visual>

File: elektron_description/robots/elektron_NoLaser_Tower-kinect.urdf.xacro (robot description, xacro)
@@ -34,5 +34,5 @@
 			<geometry>
 				<!--<box size="0.38 0.28 0.20" />-->
-				<mesh filename="package://elektron_description/meshes/elektron_body.dae"/>
+				<mesh filename="package://elektron_description/meshes/base/elektron_body.dae"/>
 			</geometry>
 		</visual>

File: elektron_description/robots/elektron_NoLaser_Tower-rgb.urdf.xacro (robot description, xacro)
@@ -34,5 +34,5 @@
 			<geometry>
 				<!--<box size="0.38 0.28 0.20" />-->
-				<mesh filename="package://elektron_description/meshes/elektron_body.dae"/>
+				<mesh filename="package://elektron_description/meshes/base/elektron_body.dae"/>
 			</geometry>
 		</visual>

Commit message: need testing

File: elektron_description/robots/elektron_Laser_NoTower.urdf.xacro (robot description, xacro)
@@ -5,9 +5,8 @@
 	xmlns:interface="http://playerstage.sourceforge.net/gazebo/xmlschema/#interface">
 	<property name="M_PI" value="3.14159"/>
-	<property name="elektron_control_input" value="pid" /> <!-- diff_drive_controller | pid -->
+	<property name="elektron_control_input" value="1" /> <!-- 0 = diff_drive_controller | 1 = pid -->
 	<property name="base_size_x" value="0.38" />
 	<property name="base_size_y" value="0.28" />
 	<property name="base_size_z" value="0.18" />
-	<xacro:arg name="use_sim" default="true" />
 	<property name="wheel_radius" value="0.05" />
 	<property name="wheel_length" value="0.02" />
@@ -15,15 +14,15 @@
 	<!-- INCLUDE SICK LMX100 LASER -->
 	<xacro:include filename="$(find elektron_description)/urdf/sensors/sick_laser_lmx_100.urdf" />
-	<!-- INCLUDE KINECT -->
+	<!-- INCLUDE KINECT
 	<xacro:include filename="$(find elektron_description)/urdf/sensors/kinect.urdf.xacro"/>
+	-->
 	<!-- INCLUDE TOWER
-	<xacro:include filename="$(find elektron_description)/urdf/tower/tower.urdf.xacro"/>-->
-  	<!-- include calibrated params -->
+	<xacro:include filename="$(find elektron_description)/urdf/tower/tower.urdf.xacro"/>
+  	-->
+	<!-- include calibrated params -->
     <xacro:include filename="$(find elektron_description)/urdf/elektron_properties.urdf.xacro"/>
-  	<!-- include gazebo control -->
-	<xacro:if value="$(arg use_sim)">
-		<xacro:include filename="$(find elektron_gazebo)/urdf/elektron_gazebo_control.urdf.xacro"/>
-		<!--<xacro:include filename="$(find elektron_gazebo)/urdf/tower_gazebo_control.urdf.xacro"/>-->
-	</xacro:if>
+	<!-- include gazebo control -->
+		<xacro:include filename="$(find elektron_control)/urdf/elektron_control.urdf.xacro"/>
+		<xacro:include filename="$(find elektron_control)/urdf/tower_control.urdf.xacro"/>
 	<!-- ROBOT BASE DEFINITION -->
 	<link name="base_link">
@@ -50,7 +49,7 @@
 		</collision>
 	</link>
-	<!-- WHEELS MACRO -->
-	<xacro:macro name="erratic_wheel" params="suffix parent reflect offset m mimic">
-			<joint name="${parent}_${suffix}_wheel_joint" type="continuous">
+<!-- WHEELS MACRO -->
+	<xacro:macro name="erratic_wheel" params="suffix parent reflect offset m mimic mimic_wheel">
+			<joint name="${parent}_${suffix}_wheel_joint" type="fixed">
 				<origin xyz="${offset} ${reflect*caster_wheel_offset_y} ${wheel_radius}" rpy="0	0 0"/>
 				<axis xyz="0 1 0" />
@@ -61,9 +60,6 @@
 				<child link="${parent}_${suffix}_wheel_link" />
 	 			<dynamics damping="0.0" friction="0.0"/>
-	 			<xacro:if value="${mimic == 'left'}">
-		 			<mimic joint="${parent}_${mimic}_wheel_joint"/>
-				</xacro:if>
-	 			<xacro:if value="${mimic == 'right'}">
-		 			<mimic joint="${parent}_${mimic}_wheel_joint"/>
+	 			<xacro:if value="${mimic}">
+		 			<mimic joint="${parent}_${mimic_wheel}_wheel_joint"/>
 				</xacro:if>
 			</joint>
@@ -99,12 +95,12 @@
 	</xacro:macro>
 	<!-- WHEELS DEFINITION -->
-	<xacro:erratic_wheel suffix="left" parent="base_link" reflect="1" offset="0" m="0.900" mimic="none"/>
-	<xacro:erratic_wheel suffix="left_front" parent="base_link" reflect="1" offset="0.15" m="0" mimic="left"/>
-	<xacro:erratic_wheel suffix="left_rear" parent="base_link" reflect="1" offset="-0.15" m="0" mimic="left"/>
-	<xacro:erratic_wheel suffix="right" parent="base_link" reflect="-1" offset="0" m="0.900" mimic="none"/>
+	<xacro:erratic_wheel suffix="left" parent="base_link" reflect="1" offset="0" m="0.900" mimic="0" mimic_wheel="left"/>
+	<xacro:erratic_wheel suffix="left_front" parent="base_link" reflect="1" offset="0.15" m="0" mimic="1" mimic_wheel="left"/>
+	<xacro:erratic_wheel suffix="left_rear" parent="base_link" reflect="1" offset="-0.15" m="0" mimic="1" mimic_wheel="left"/>
+	<xacro:erratic_wheel suffix="right" parent="base_link" reflect="-1" offset="0" m="0.900" mimic="0" mimic_wheel="left"/>
 	<xacro:erratic_wheel suffix="right_front" parent="base_link" reflect="-1" offset="0.15"
-		m="0" mimic="right"/>
-	<xacro:erratic_wheel suffix="right_rear" parent="base_link" reflect="-1" offset="-0.15"	m="0" mimic="right"/>
-<!-- ADD KINECT -->
+		m="0" mimic="1" mimic_wheel="right" />
+	<xacro:erratic_wheel suffix="right_rear" parent="base_link" reflect="-1" offset="-0.15"	m="0" mimic="1" mimic_wheel="right"/>
+<!-- ADD KINECT
     <joint name="bottom_kinect_joint" type="fixed">
       <origin xyz="${kinect_px} ${kinect_py} ${kinect_pz}" rpy="${kinect_or} ${kinect_op} ${kinect_oy}"/>
@@ -114,12 +110,13 @@
     <link name="bottom_kinect_link"/>
 	<sensor_kinect parent="bottom_kinect_link" id="bottom"/>
-	<!-- ADD TOWER -->
-	<!-- <elektron_tower parent="base_link" camera_type="rgb_camera" id="1"/> camera_type avaliable: kinect | rgb_camera
-	<tower_PID_control_gazebo/>-->
+ADD TOWER
+	<elektron_tower parent="base_link" camera_type="0" id="1"/> camera_type avaliable: 1 = kinect | 0 = rgb_camera
+	<tower_PID_control_gazebo/>
+-->
 	<!-- SET gazebo-ROS CONTROL -->
-	<xacro:if value="${elektron_control_input == 'pid'}">
+	<xacro:if value="${elektron_control_input}">
 		<elektron_PID_control_gazebo/>
 	</xacro:if>
-	<xacro:if value="${elektron_control_input == 'diff_drive_controller'}">
+	<xacro:unless value="${elektron_control_input}">
 		<gazebo>
 		<plugin name="differential_drive_controller" filename="libgazebo_ros_diff_drive.so">
@@ -137,4 +134,4 @@
 		</plugin>
 	</gazebo>
-	</xacro:if>
+	</xacro:unless>
 </robot>
