Commit message: add tower link mesh

File: elektron_description/urdf/elektron_properties.urdf.xacro (robot description, xacro)
@@ -19,5 +19,5 @@
      (currently in development and awaiting feedback)
    -->
-	<property name="kinect_px" value="0.1" />
+	<property name="kinect_px" value="-0" />
 	<property name="kinect_py" value="0.0" />  <!-- Y varies for different configurations. get sets in sensors_urdf -->
 	<property name="kinect_pz" value="0.45"/>
@@ -25,5 +25,5 @@
 	<property name="kinect_op" value="0" />
 	<property name="kinect_oy" value="0" />
-	<property name="head_base_px" value="0.1" />
+	<property name="head_base_px" value="0" />
 	<property name="head_base_py" value="0.0" />
 	<property name="head_base_pz" value="0.75"/>
@@ -31,7 +31,7 @@
 	<property name="head_base_op" value="0" />
 	<property name="head_base_oy" value="0" />
-	<property name="high_kinect_base_px" value="0" />
+	<property name="high_kinect_base_px" value="-0.05" />
 	<property name="high_kinect_base_py" value="0" />
-	<property name="high_kinect_base_pz" value="1.2" />
+	<property name="high_kinect_base_pz" value="1.15" />
 	<property name="high_kinect_base_or" value="0" />
 	<property name="high_kinect_base_op" value="0" />

File: elektron_description/urdf/tower/tower.urdf.xacro (robot description, xacro)
@@ -29,4 +29,10 @@
 		     <inertia ixx="1"  ixy="0"  ixz="0" iyy="1" iyz="0" izz="1" />
    		</inertial>
+      	<visual>
+	       <origin xyz="0 0 0" rpy="0 0 ${M_PI/2}"/>
+		<geometry>
+		 <mesh filename="package://elektron_description/meshes/base/tower.dae"/>
+		</geometry>
+      </visual>
 	</link>
     <joint name="head_yaw_fixed_joint_${id}" type="fixed">

Commit message: real elektron tf fix, new tower mesh

File: elektron_description/urdf/elektron_properties.urdf.xacro (robot description, xacro)
@@ -31,5 +31,5 @@
 	<property name="head_base_op" value="0" />
 	<property name="head_base_oy" value="0" />
-	<property name="high_kinect_base_px" value="-0.05" />
+	<property name="high_kinect_base_px" value="-0.15" />
 	<property name="high_kinect_base_py" value="0" />
 	<property name="high_kinect_base_pz" value="1.15" />

File: elektron_description/urdf/tower/tower.urdf.xacro (robot description, xacro)
@@ -132,5 +132,5 @@
 		<elektron_rgb_camera parent="head_end_link_${id}" id="head"/>
     <joint name="camera_rgb_${id}" type="fixed">
-      <origin xyz="0.0 0.0 0.0" rpy="0 -${M_PI/2} ${M_PI/2}"/>
+      <origin xyz="0.0 0.0 0.0" rpy="0 0 0"/>
       <parent link="camera_optical_link_head"/>
       <child link="rgb_head_${id}"/>
